File: memory_module/memory_module.kicad_pcb (KiCad board)
At the start: 2 copper layers, 100 x 100 mm, 174 parts, among them J1 Conn_01x06_Pin, J2 Conn_01x08_Pin, SW1 SW_DIP_x08, SW10 SW_DIP_x08, SW11 SW_DIP_x08, SW12 SW_DIP_x08, SW13 SW_DIP_x08, SW14 SW_DIP_x08, SW15 SW_DIP_x08, SW16 SW_DIP_x08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

Commit message: パスコンwip
Connections:
- J1 pad 6: GND -> +5V
- U1 pad 8: GND -> +5V
- U2 pad 4: GND -> +5V
- U2 pad 5: GND -> +5V
- U2 pad 8: GND -> +5V
- U3 pad 1: GND -> +5V
- U3 pad 10: GND -> +5V
- U3 pad 19: GND -> +5V
Routing:
- net GND: track 141.9 -> 0.00 mm
- net +5V: track 120.9 -> 262.8 mm
- added copper zone on B.Cu, net +5V
- added copper zone on F.Cu, net +5V
- removed copper zone on B.Cu, net GND
- removed copper zone on F.Cu, net GND

Commit message: パスコン追加
Parts:
- added C1: 0.1μF, Capacitor_THT:C_Disc_D4.3mm_W1.9mm_P5.00mm, F.Cu at (41.3, 123.2)
- added C2: 0.1μF, Capacitor_THT:C_Disc_D4.3mm_W1.9mm_P5.00mm, F.Cu at (64.1, 123.2)
- added C3: 0.1μF, Capacitor_THT:C_Disc_D4.3mm_W1.9mm_P5.00mm, F.Cu at (138.4, 131.4)
- moved R9 2.11 mm to (108.2, 132.7)
- moved U3 1.42 mm to (135.9, 123.8)
- moved U2 1.27 mm to (66.7, 130.8)
Connections:
- J1 pad 6: +5V -> GND
- U1 pad 8: +5V -> GND
- U2 pad 4: +5V -> GND
- U2 pad 5: +5V -> GND
- U2 pad 8: +5V -> GND
- U3 pad 1: +5V -> GND
- U3 pad 10: +5V -> GND
- U3 pad 19: +5V -> GND
Routing:
- net +5V: track 262.8 -> 136.5 mm
- net GND: track 0.00 -> 85.9 mm, vias 0 -> 12
- net A0: track 41.9 -> 31.9 mm
- net A1: track 44.2 -> 37.9 mm
- net A2: track 45.6 -> 43.3 mm
- net Net-(D105-K): track 36.8 -> 38.3 mm
- net Net-(D100-K): track 38.5 -> 39.7 mm
- net Net-(D140-K): track 85.4 -> 84.2 mm
- net Net-(D121-K): track 62.8 -> 61.6 mm
- net Net-(D113-K): track 33.0 -> 31.7 mm
- net Net-(U3-A7): track 393.6 -> 394.8 mm
- net Net-(U3-A6): track 392.8 -> 393.9 mm
- net Net-(U3-A4): track 392.3 -> 393.4 mm
- net Net-(U3-A2): track 391.2 -> 392.3 mm
- net Net-(U3-A1): track 390.9 -> 392.1 mm
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- added copper zone on B.Cu, net GND
- added copper zone on F.Cu, net GND
- removed copper zone on B.Cu, net +5V
- removed copper zone on F.Cu, net +5V
Other:
- board text added: "+5V"
- board text removed: "5V"
