File: clock_module/clock_module.kicad_sch (KiCad schematic)
At the start: 53 parts, among them J1 USB_C_Receptacle_PowerOnly_6P, SW1 SW_SPST, SW2 SW_Push, SW3 SW_SPDT, SW4 SW_SPDT, U1 74HC14, U10 74HC74, U11 SN74HC10N, U2 74HC161N, U3 74HC161N, U4 74HC161N, U5 74HC161N, U6 74HC153N, U7 74HC153N, U8 CD74HC283E, U9 SN74HC32N

Commit message: 回路図いったん完成
Parts:
- removed U11: SN74HC10N, N14, symbol 74hc10:SN74HC10N
- removed U8: CD74HC283E, footprint_library:74hc283, symbol 74hc283:CD74HC283E
- removed U9: SN74HC32N, footprint_library:74hc32, symbol 74hc32:SN74HC32N
- added J2: Conn_01x06_Socket, symbol Connector:Conn_01x06_Socket
- added J3: Conn_01x08_Socket, symbol Connector:Conn_01x08_Socket
- added R19, R20, R21, R22: R, symbol Device:R
- added SW5: SW_DIP_x04, symbol Switch:SW_DIP_x04
- added U11: 74HC10, footprint_library:74hc10, symbol 74xx:74LS10
- added U8: 74HC283, footprint_library:74hc283, symbol 74xx:74LS283
- added U9: 74HC32, footprint_library:74hc32, symbol 74xx:74LS32
Connections:
- net +5V: now also U10.10 (~{S}), J2.5 (Pin_5), SW5.5, SW5.6, SW5.7, SW5.8, U11.1, U11.10, U11.14 (VCC), U11.9, U8.16 (VCC), U9.14 (VCC)
- net A0: now also J2.1 (Pin_1)
- net A1: now also J2.2 (Pin_2)
- net A2: now also J2.3 (Pin_3)
- net A3: now also J2.4 (Pin_4)
- net CLOCK: now also U10.11 (C)
- net GND: now also U10.1 (~{R}), U10.2 (D), U10.3 (C), U10.4 (~{S}), J2.6 (Pin_6), R19.2, R20.2, R21.2, R22.2, U11.7 (GND), U8.7 (C0), U8.8 (GND), U9.7 (GND); no longer U10.10 (~{S}), U10.11 (C), U10.12 (D), U10.13 (~{R})
- net RESET: now also U10.13 (~{R})
- net at U2.3 (D0), U3.3 (D0), U4.3 (D0)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: now also U8.4 (S1)
- net at U2.4 (D1), U3.4 (D1), U4.4 (D1)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: now also U8.1 (S2)
- net at U2.5 (D2), U3.5 (D2), U4.5 (D2)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: now also U8.13 (S3)
- net at U2.6 (D3), U3.6 (D3), U4.6 (D3)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: now also U8.10 (S4)
- net at U4.9 (PE*): now also U11.12
- net at U7.12 (2I2): now also R22.1, SW5.4
- net SELECT B: now reaches U7.14 (SO)
- net SELECT B: now also U6.14 (SO), U9.11
- net D5: now reaches U7.2 (S1)
- net D5: now also U6.2 (S1), J3.6 (Pin_6)
- net at U7.4 (1I2): now also R21.1, SW5.3
- net at U7.7 (1Y): now also U8.14 (A3)
- net at U7.9 (2Y): now also U8.12 (A4)
- net at U6.12 (2I2): now also R20.1, SW5.2
- net at U6.4 (1I2): now also R19.1, SW5.1
- net at U6.7 (1Y): now also U8.5 (A1)
- net at U6.9 (2Y): now also U8.3 (A2)
- net at U2.9 (PE*): now also U9.3
- net at U3.9 (PE*): now also U9.6
- net at U10.8 (~{Q}): now also U9.9
- net at U5.9 (PE*): now also U11.6
- new net: U11.5, U9.8
- new net: U10.12 (D), U8.9 (C4)
- new net: U11.2, U11.8, U9.4
- new net D0: J3.1 (Pin_1), U8.6 (B1)
- new net D1: J3.2 (Pin_2), U8.2 (B2)
- new net D2: J3.3 (Pin_3), U8.15 (B3)
- new net D3: J3.4 (Pin_4), U8.11 (B4)
- new net D4: J3.5 (Pin_5), U9.10, U9.13
- new net D6: J3.7 (Pin_7), U11.11, U11.3, U9.1
- new net D7: J3.8 (Pin_8), U11.13, U11.4, U9.12, U9.2, U9.5
- no-connect marks 8 -> 9
Other:
- moved on the sheet: D1, D2, D3, D4, R15, R16, R17, R18, U10A, U10C, U1F, U1G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
