File: clock_module/clock_module.kicad_pcb (KiCad board)
At the start: 2 copper layers, 100 x 100 mm, 60 parts, among them J1 USB_C_Receptacle_PowerOnly_6P, J2 Conn_01x06_Socket, J3 Conn_01x08_Socket, SW1 SW_SPST, SW2 SW_Push, SW3 SW_SPDT, SW4 SW_SPDT, SW5 SW_DIP_x04, U1 74HC14, U10 74HC74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

Commit message: add: 配線
Parts:
- moved D1 81.2 mm to (135.3, 59.7)
- moved R15 80.9 mm to (135.3, 54.4)
- moved D2 80.6 mm to (141.6, 59.7)
- moved R16 80.2 mm to (141.6, 54.4)
- moved D3 79.9 mm to (148.0, 59.7)
- moved R17 79.4 mm to (148.0, 54.4)
- moved D4 79.3 mm to (154.3, 59.7)
- moved R18 78.7 mm to (154.3, 54.4)
- moved R22 16.3 mm to (181.0, 132.1)
- moved R21 15.8 mm to (184.2, 132.1)
- moved R20 15.5 mm to (187.3, 132.1)
- moved R19 15.5 mm to (190.5, 132.1)
- moved C7 2.15 mm to (166.4, 66.0)
- moved U6 2.15 mm to (158.8, 68.6)
- moved C8 0.77 mm to (179.2, 66.0)
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Routing:
- net +5V: track 333.0 -> 442.2 mm
- net D7: track 0.00 -> 101.0 mm
- net D6: track 0.00 -> 97.4 mm, vias 0 -> 2
- net D4: track 0.00 -> 95.9 mm
- net Net-(U6-I2a): track 0.00 -> 84.4 mm, vias 0 -> 2
- net SELECT A: track 0.00 -> 82.0 mm
- net R_A2: track 0.00 -> 76.7 mm, vias 0 -> 1
- net R_A3: track 0.00 -> 74.3 mm, vias 0 -> 1
- net Net-(U6-I2b): track 0.00 -> 74.2 mm, vias 0 -> 2
- net Net-(U7-I2a): track 0.00 -> 70.9 mm
- net Net-(U2-D2): track 36.0 -> 104.7 mm, vias 0 -> 3
- net R_A0: track 0.00 -> 67.9 mm, vias 0 -> 2
- net R_B3: track 0.00 -> 65.6 mm, vias 0 -> 4
- net GND: track 201.5 -> 266.9 mm, vias 0 -> 17
- net R_A1: track 0.00 -> 65.0 mm, vias 0 -> 1
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- added copper zone on B.Cu, net GND
- added copper zone on F.Cu, net GND
